Commit message: Completed working the basic of working with parameters for both cpp and python.

File: install/arduino_description/share/arduino_description/urdf/arduino_urldf.xacro (robot description, xacro)
@@ -22,5 +22,5 @@
     <link name="base_plate">
         <visual>
-            <origin rpy="0 0 0" xyz="0 -0.2 0"/>
+            <origin rpy="0 0 0" xyz="0 0 -0.3101"/>
             <geometry>
                 <mesh filename="package://arduino_description/meshes/base/MountPlate_BasePlate.stl" scale="0.01 0.01 0.01" />
@@ -35,3 +35,25 @@
         <limit lower="-${PI/2}" upper="${PI/2}" effort="${effort}" velocity="${velocity}" />
     </joint>
+    <link name="forward_drive_arm">
+        <visual>
+            <origin xyz="0 0 0" rpy="0.39 - 0" />
+            <geometry>
+                <mesh filename="package://package_name/meshes/mesh.stl" />
+            </geometry>
+            <material name="material_name">
+                <color rgba="1 1 1 1" />
+            </material>
+        </visual>
+        <collision>
+            <origin xyz="0 0 0" rpy="0 0 0" />
+            <geometry>
+                <mesh filename="package://package_name/meshes/mesh.stl" />
+            </geometry>
+        </collision>
+        <inertial>
+            <mass value="1.0" />
+            <origin xyz="0 0 0" />
+            <inertia ixx="1.0" ixy="0.0" ixz="0.0" iyy="1.0" iyz="0.0" izz="1.0" />
+        </inertial>
+    </link>
 </robot>

File: src/arduino_description/urdf/arduino_urldf.xacro (robot description, xacro)
@@ -35,3 +35,25 @@
         <limit lower="-${PI/2}" upper="${PI/2}" effort="${effort}" velocity="${velocity}" />
     </joint>
+    <link name="forward_drive_arm">
+        <visual>
+            <origin xyz="0 0 0" rpy="0.39 - 0" />
+            <geometry>
+                <mesh filename="package://package_name/meshes/mesh.stl" />
+            </geometry>
+            <material name="material_name">
+                <color rgba="1 1 1 1" />
+            </material>
+        </visual>
+        <collision>
+            <origin xyz="0 0 0" rpy="0 0 0" />
+            <geometry>
+                <mesh filename="package://package_name/meshes/mesh.stl" />
+            </geometry>
+        </collision>
+        <inertial>
+            <mass value="1.0" />
+            <origin xyz="0 0 0" />
+            <inertia ixx="1.0" ixy="0.0" ixz="0.0" iyy="1.0" iyz="0.0" izz="1.0" />
+        </inertial>
+    </link>
 </robot>
